File: SSI2131_Card/SSI2131_Edge_Card.kicad_pcb (KiCad board)
At the start: 2 copper layers, 70 parts, among them Q1 2N3906, Q2 2N3906, U1 SSI2131, U2 SSI2131, U3 LM4040DBZ-2.5, U4 LM13700, U5 OPA1678, U6 CD4066BM, U7 OPA1678, U8 OPA1678

Commit message: adjusted PCB layout for new haiarchy
Parts:
- removed C1, C5: 220nF, Capacitor_SMD:C_0603_1608Metric
- removed C10, C19: 470nF, Capacitor_SMD:C_0603_1608Metric
- removed C11, C12, C13, C14, C15, C16, C17, C20, C21: 0.1uf, Capacitor_SMD:C_0603_1608Metric
- removed C18, C9: 1nF, Capacitor_SMD:C_0603_1608Metric
- removed C2, C3: 10n, Capacitor_SMD:C_0603_1608Metric
- removed C4, C6: 3.9nf, Capacitor_THT:C_Rect_L7.2mm_W2.5mm_P5.00mm_FKS2_FKP2_MKS2_MKP2
- removed C7, C8: 1uf, Capacitor_SMD:C_0805_2012Metric
- removed D1, D2: 1N4148W, Diode_SMD:D_SOD-123
- removed Q1, Q2: 2N3906, Package_TO_SOT_THT:TO-92_Inline
- removed R1, R9: 100k, Resistor_SMD:R_0603_1608Metric
- removed R10, R2: 5k, Potentiometer_THT:Potentiometer_Bourns_3296W_Vertical
- removed R11, R15, R23, R3, R8: 10k, Resistor_SMD:R_0603_1608Metric
- removed R12, R4: 680, Resistor_SMD:R_0603_1608Metric
- removed R13, R5: 20k, Resistor_SMD:R_0603_1608Metric
- removed R14: 2k, Resistor_SMD:R_0805_2012Metric
- removed R16, R24: 2.5k, Resistor_SMD:R_0603_1608Metric
- removed R17, R26: 6.8k, Resistor_SMD:R_0603_1608Metric
- removed R18, R29: 33k, Resistor_SMD:R_0603_1608Metric
- removed R19, R30: 120k, Resistor_SMD:R_0603_1608Metric
- removed R20, R31: 3.9k, Resistor_SMD:R_0603_1608Metric
- removed R21, R22, R25, R27, R28, R32, R33, R34, R35: 1k, Resistor_SMD:R_0603_1608Metric
- removed R6: 267k, Resistor_THT:R_Axial_DIN0207_L6.3mm_D2.5mm_P5.08mm_Vertical
- removed R7: 4.3k, Resistor_SMD:R_0603_1608Metric
- removed TP1: 2V5 TP, TestPoint:TestPoint_Pad_1.0x1.0mm
- removed TP2: PMOD_TP, TestPoint:TestPoint_Pad_1.0x1.0mm
- removed U1, U2: SSI2131, Package_SO:STC_SOP-16_3.9x9.9mm_P1.27mm
- removed U3: LM4040DBZ-2.5, Package_TO_SOT_SMD:SOT-23
- removed U4: LM13700, Package_SO:SOIC-16_3.9x9.9mm_P1.27mm
- removed U5, U7, U8: OPA1678, Package_SO:SOIC-8_3.9x4.9mm_P1.27mm
- removed U6: CD4066BM, Package_SO:SOIC-14_3.9x8.7mm_P1.27mm
