File: SSI2131_Card/SSI2131_Edge_Card.kicad_sch (KiCad schematic)
At the start: 62 parts, among them Q1 2N3906, Q2 2N3906, U1 CD4066BM, U2 OPA1678, U3 OPA1678, U4 LM13700, U5 SSI2131, U6 SSI2131, U7 LM4040DBZ-2.5

Commit message: Aded Heiarchy in Kicad, adjusted overall VCA design
Parts:
- removed C1, C3: 470nF, Capacitor_SMD:C_0603_1608Metric, symbol Device:C
- removed C13, C14, C15, C16, C17, C18, C19: 0.1uf, Capacitor_SMD:C_0603_1608Metric, symbol Device:C
- removed C5, C6: 1nF, Capacitor_SMD:C_0603_1608Metric, symbol Device:C
- removed D1, D2: 1N4148W, Diode_SMD:D_SOD-123, symbol Diode:1N4148W
- removed Q1, Q2: 2N3906, Package_TO_SOT_THT:TO-92_Inline, symbol Transistor_BJT:2N3906
- removed R10, R13, R14, R15: 1k, Resistor_SMD:R_0603_1608Metric, symbol Device:R
- removed R12, R8: 2.5k, Resistor_SMD:R_0603_1608Metric, symbol Device:R
- removed R17, R18: 6.8k, Resistor_SMD:R_0603_1608Metric, symbol Device:R
- removed R19, R21: 33k, Resistor_SMD:R_0603_1608Metric, symbol Device:R
- removed R2, R4: 120k, Resistor_SMD:R_0603_1608Metric, symbol Device:R
- removed R3, R6: 10k, Resistor_SMD:R_0603_1608Metric, symbol Device:R
- removed R7, R9: 3.9k, Resistor_SMD:R_0603_1608Metric, symbol Device:R
- removed TP1: 2V5 TP, TestPoint:TestPoint_Pad_1.0x1.0mm, symbol Connector:TestPoint
- removed U1: CD4066BM, Package_SO:SOIC-14_3.9x8.7mm_P1.27mm, symbol 4xxx:4066
- removed U2, U3: OPA1678, Package_SO:SOIC-8_3.9x4.9mm_P1.27mm, symbol Amplifier_Operational:OPA1678
- removed U4: LM13700, Package_SO:SOIC-16_3.9x9.9mm_P1.27mm, symbol Amplifier_Operational:LM13700
Other:
- added sheet Pitch and PWM modulation (Pitch_PWM_mod.kicad_sch)
- note removed: "2.5V DAC Input"
- note removed: "2.5Vpp Input"

Commit message: Added pin lables and added VCOs into their own heiarchy sheets
Parts:
- removed C10, C9: 3.9nf, Capacitor_THT:C_Rect_L7.2mm_W2.5mm_P5.00mm_FKS2_FKP2_MKS2_MKP2, symbol Device:C_US
- removed C2, C4: 220nF, Capacitor_SMD:C_0603_1608Metric, symbol Device:C
- removed C7, C8: 10n, Capacitor_SMD:C_0603_1608Metric, symbol Device:C
- removed R1, R11: 680, Resistor_SMD:R_0603_1608Metric, symbol Device:R
- removed R16, R5: 20k, Resistor_SMD:R_0603_1608Metric, symbol Device:R
- removed R20, R28: 5k, Potentiometer_THT:Potentiometer_Bourns_3296W_Vertical, symbol Device:R_Potentiometer
- removed R22, R26, R29: 10k, Resistor_SMD:R_0603_1608Metric, symbol Device:R
- removed R23, R30: 100k, Resistor_SMD:R_0603_1608Metric, symbol Device:R
- removed R24: 4.3k, Resistor_SMD:R_0603_1608Metric, symbol Device:R
- removed R25: 267k, Resistor_THT:R_Axial_DIN0207_L6.3mm_D2.5mm_P5.08mm_Vertical, symbol Device:R_US
- removed U5, U6: SSI2131, Package_SO:STC_SOP-16_3.9x9.9mm_P1.27mm, symbol Sound_Semiconductor:SSI2131
- renumbered C11 to C7, C12 to C8, R27 to R14, TP2 to TP1, U7 to U3
Other:
- added sheet OSC A (OSC_A.kicad_sch)
- added sheet OSC B (OSC_B.kicad_sch)
- sheet Pitch and PWM modulation ports: added PMOD_AMT, PMOD_EN, PMOD_IN, PWM_MOD_AMOUNT, PWM_MOD_EN, PWM_MOD_IN; removed none
