File: STM32G474RE_TB/DacBuffers.kicad_sch (KiCad schematic)
At the start: 33 parts, among them U11 OPA1678, U12 OPA1678, U13 OPA1678, U14 OPA1678

Commit message: Added MOSFET template with led for debug or other functions
Parts:
- renumbered C36 to C24, C34 to C25, C32 to C26, C30 to C27, C24 to C28, C37 to C29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
