File: Dev_Hardware/QFN_Practice/Mcu_supp_sch.kicad_sch (KiCad schematic)
At the start: 5 parts, among them J2 FTSH-105-01-X-DV-K-X, SW1 SW_Push, SW3 SW_Push

Commit message: finished routing for all but power regulation and GPIO
Connections:
- net nRST: no longer R2.2, SW3.2
- net ISP renamed m_ISP
- new net m_nRST: R2.2, SW3.2
Changed lines of the file:
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@@
 		)
 	)
-	(hierarchical_label "nRST"
+	(hierarchical_label "m_nRST"
 		(shape input)
 		(at 36.83 74.93 180)
@@
 		)
 	)
-	(hierarchical_label "ISP"
+	(hierarchical_label "m_ISP"
 		(shape input)
 		(at 39.37 30.48 180)
